File: lighting-controller/board/swampgas.sch (KiCad schematic (older format))
At the start: 19 parts, among them J1 LiPo 3.7V, J2 NeoPixel, J3 Dome, SW1 SW_DIP_x08, U1 Adafruit Trinket M0, U2 CD4512BE

Commit message: Version 1.1 - flying Oct 30 2021!
Parts:
- J1: symbol B2B-PH-SM4-TB_LF__SN_:B2B-PH-SM4-TB(LF)(SN) -> swampgas-rescue:B2B-PH-SM4-TB(LF)(SN)-B2B-PH-SM4-TB_LF__SN_
Changed lines of the file:
@@
 $EndComp
 $Comp
-L B2B-PH-SM4-TB_LF__SN_:B2B-PH-SM4-TB(LF)(SN) J1
+L swampgas-rescue:B2B-PH-SM4-TB(LF)(SN)-B2B-PH-SM4-TB_LF__SN_ J1
 U 1 1 5F400C6F
 P 1350 2450
